Commit message: updated

File: robot_description/urdf/gazebo.urdf.xacro (robot description, xacro)
@@ -1,23 +1,26 @@
 <?xml version="1.0"?>
 <robot xmlns:xacro="http://www.ros.org/wiki/xacro">
+    <gazebo reference="imu_link">
+        <sensor name="imu_sensor" type="imu">
+            <gz_frame_id>robot/imu_link</gz_frame_id>
+            <update_rate>50</update_rate>
+            <visualize>false</visualize>
+            <topic>imu</topic>
+            <always_on>false</always_on>
+        </sensor>
+    </gazebo>
+    <link name="imu_link" />
+    <joint name="imu_link_joint" type="fixed">
+        <parent link="base_link"/>
+        <child link="imu_link"/>
+    </joint>
     <gazebo>
-        <!--plugin
-            filename="gz-sim-pose-publisher-system"
-            name="gz::sim::systems::PosePublisher">
-            <publish_link_pose>true</publish_link_pose>
-            <use_pose_vector_msg>true</use_pose_vector_msg>
-            <static_publisher>true</static_publisher>
-            <static_update_frequency>1</static_update_frequency>
-        </plugin-->
-        <!--plugin
-            filename="gz-sim-odometry-publisher-system"
-            name="gz::sim::systems::OdometryPublisher">
-            <odom_frame>robot/odom</odom_frame>
-            <robot_base_frame>robot/base_link</robot_base_frame>
-            <odom_publish_frequency>50</odom_publish_frequency>
-        </plugin-->
         <plugin
             filename="gz-sim-joint-state-publisher-system"
             name="gz::sim::systems::JointStatePublisher">
+        </plugin>
+        <plugin
+            filename="gz-sim-imu-system"
+            name="gz::sim::systems::Imu">
         </plugin>
         <plugin
@@ -27,7 +30,18 @@
             <right_joint>right_wheel_joint</right_joint>
             <child_frame_id>robot/base_link</child_frame_id>
-            <wheel_separation>0.291</wheel_separation>
+            <wheel_separation>0.11</wheel_separation>
             <wheel_radius>0.033</wheel_radius>
-            <odom_publish_frequency>10</odom_publish_frequency>
+            <odom_publish_frequency>50</odom_publish_frequency>
+            <min_velocity>-1.0</min_velocity>
+            <max_velocity>1.0</max_velocity>
+            <min_acceleration>-0.3</min_acceleration>
+            <max_acceleration>0.3</max_acceleration>
+            <min_angular_acceleration>-1.0</min_angular_acceleration>
+            <max_angular_acceleration>1.0</max_angular_acceleration>
+        </plugin>
+        <plugin
+            filename="gz-sim-sensors-system"
+            name="gz::sim::systems::Sensors">
+            <render_engine>ogre2</render_engine>
         </plugin>
     </gazebo>

File: robot_description/urdf/robot.urdf.xacro (robot description, xacro)
@@ -2,19 +2,20 @@
 <robot name='robot' xmlns:xacro="http://ros.org/wiki/xacro">
     <xacro:include filename="$(find robot_description)/urdf/gazebo.urdf.xacro" />
-    <!--xacro:include filename="$(find robot_description)/urdf/lidar.urdf.xacro" /-->
-    <!--xacro:include filename="$(find robot_description)/urdf/depth.urdf.xacro" /-->
-    <xacro:property name="chassis_length" value="0.335"/>
-    <xacro:property name="chassis_width" value="0.265"/>
-    <xacro:property name="chassis_height" value="0.138"/>
+    <xacro:include filename="$(find robot_description)/urdf/lidar.urdf.xacro" />
+    <xacro:include filename="$(find robot_description)/urdf/depth.urdf.xacro" />
+    <xacro:property name="M_PI" value="3.1415926535897931" />
+    <xacro:property name="chassis_length" value="0.176"/>
+    <xacro:property name="chassis_width" value="0.13"/>
+    <xacro:property name="chassis_height" value="0.069"/>
     <xacro:property name="wheel_radius" value="0.033"/>
-    <xacro:property name="wheel_thickness" value="0.026"/>
-    <xacro:property name="wheel_mass" value="0.05"/>
-    <xacro:property name="wheel_offset_x" value="0.226"/>
-    <xacro:property name="wheel_offset_y" value="0.1485"/>
+    <xacro:property name="wheel_thickness" value="0.018"/>
+    <xacro:property name="wheel_mass" value="0.2"/>
+    <xacro:property name="wheel_offset_x" value="0.0375"/>
+    <xacro:property name="wheel_offset_y" value="0.055"/>
     <xacro:property name="wheel_offset_z" value="0.01"/>
-    <xacro:property name="caster_wheel_radius" value="0.01"/>
+    <xacro:property name="caster_wheel_radius" value="0.024"/>
     <xacro:property name="caster_wheel_mass" value="0.01"/>
-    <xacro:property name="caster_wheel_offset_x" value="0.075"/>
-    <xacro:property name="caster_wheel_offset_z" value="${wheel_offset_z - wheel_radius + caster_wheel_radius}"/>
+    <xacro:property name="caster_wheel_offset_x" value="0.08"/>
+    <xacro:property name="caster_wheel_offset_z" value="-0.05"/>
     <xacro:property name="mass" value="1.0"/>
     <material name="white">
@@ -33,39 +34,34 @@
         <color rgba="1 0 0 1"/>
     </material>
-    <link name="base_link">
-    </link>
-    <link name="base_footprint">
-    </link>
+    <link name="base_link" />
+    <link name="base_footprint" />
     <joint name="base_footprint_joint" type="fixed">
         <parent link="base_link"/>
         <child link="base_footprint"/>
-        <origin xyz="0 0 -0.138" rpy="0 0 0"/>
+        <origin xyz="0 0 -0.03" rpy="0 0 0"/>
     </joint>
     <joint name="chassis_joint" type="fixed">
         <parent link="base_link"/>
         <child link="chassis"/>
-        <origin xyz="${-wheel_offset_x} 0 ${-wheel_offset_z}"/>
+        <origin xyz="0 0 0.04" rpy="0 0 ${M_PI}"/>
     </joint>
     <link name='chassis'>
-    <inertial>
-        <origin xyz="${chassis_length/2} 0 ${chassis_height/2}" rpy="0 0 0"/>
-        <mass value="${mass}" />
-        <inertia ixx="${(1/12) * mass * (chassis_width*chassis_width+chassis_height*chassis_height)}" ixy="0.0" ixz="0.0"
-                 iyy="${(1/12) * mass * (chassis_length*chassis_length+chassis_height*chassis_height)}" iyz="0.0"
-                 izz="${(1/12) * mass * (chassis_length*chassis_length+chassis_width*chassis_width)}" />
-    </inertial>
-    <visual>
-        <origin xyz="${chassis_length/2} 0 ${chassis_height/2}"/>
-        <geometry>
-            <box size="${chassis_length} ${chassis_width} ${chassis_height}"/>
-        </geometry>
-        <material name="orange"/>
-    </visual>
-    <collision>
-        <origin xyz="${chassis_length/2} 0 ${chassis_height/2}"/>
-        <geometry>
-            <box size="${chassis_length} ${chassis_width} ${chassis_height}"/>
-        </geometry>
-    </collision>
+        <inertial>
+            <mass value="${mass}" />
+            <inertia ixx="1e-3" ixy="0.0" ixz="0.0"
+                     iyy="1e-3" iyz="0.0"
+                     izz="1e-3" />
+        </inertial>
+        <visual>
+            <geometry>
+                <mesh filename="file://$(find robot_description)/urdf/body_center_sim.stl" scale="0.001 0.001 0.001"/>
+            </geometry>
+            <material name="blue"/>
+        </visual>
+        <collision>
+            <geometry>
+                <box size="${chassis_length} ${chassis_width} ${chassis_height}"/>
+            </geometry>
+        </collision>
     </link>
     <gazebo reference="chassis">
@@ -75,11 +71,11 @@
         <parent link="base_link"/>
         <child link="left_wheel"/>
-        <origin xyz="0 ${wheel_offset_y} 0" rpy="-${pi/2} 0 0" />
-        <axis xyz="0 0 1"/>
+        <origin xyz="${wheel_offset_x} ${wheel_offset_y} 0" rpy="0 0 0" />
+        <axis xyz="0 1 0"/>
     </joint>
     <link name="left_wheel">
         <visual>
             <geometry>
-                <cylinder radius="${wheel_radius}" length="${wheel_thickness}"/>
+                <mesh filename="file://$(find robot_description)/urdf/left_tire_sim.stl" scale="0.001 0.001 0.001"/>
             </geometry>
             <material name="blue"/>
@@ -92,8 +88,8 @@
         <inertial>
             <origin xyz="0 0 0" rpy="0 0 0"/>
-            <mass value="${wheel_mass}" />
-            <inertia ixx="${(1/12) * wheel_mass * (3*wheel_radius*wheel_radius + wheel_thickness*wheel_thickness)}" ixy="0.0" ixz="0.0"
-                     iyy="${(1/12) * wheel_mass * (3*wheel_radius*wheel_radius + wheel_thickness*wheel_thickness)}" iyz="0.0"
-                     izz="${(1/2) * wheel_mass * (wheel_radius*wheel_radius)}" />
+            <mass value="2.8498940e-02" />
+            <inertia ixx="1.1175580e-05" ixy="-4.2369783e-11" ixz="-5.9381719e-09"
+                     iyy="1.1192413e-05" iyz="-1.4400107e-11"
+                     izz="2.0712558e-05" />
         </inertial>
     </link>
@@ -104,11 +100,11 @@
         <parent link="base_link"/>
         <child link="right_wheel"/>
-        <origin xyz="0 ${-wheel_offset_y} 0" rpy="${pi/2} 0 0" />
-        <axis xyz="0 0 -1"/>
+        <origin xyz="${wheel_offset_x} ${-wheel_offset_y} 0" rpy="0 0 0" />
+        <axis xyz="0 1 0"/>
     </joint>
     <link name="right_wheel">
         <visual>
             <geometry>
-                <cylinder radius="${wheel_radius}" length="${wheel_thickness}"/>
+                <mesh filename="file://$(find robot_description)/urdf/right_tire_sim.stl" scale="0.001 0.001 0.001"/>
             </geometry>
             <material name="blue"/>
@@ -121,8 +117,8 @@
         <inertial>
             <origin xyz="0 0 0" rpy="0 0 0"/>
-            <mass value="${wheel_mass}" />
-            <inertia ixx="${(1/12) * wheel_mass * (3*wheel_radius*wheel_radius + wheel_thickness*wheel_thickness)}" ixy="0.0" ixz="0.0"
-                     iyy="${(1/12) * wheel_mass * (3*wheel_radius*wheel_radius + wheel_thickness*wheel_thickness)}" iyz="0.0"
-                     izz="${(1/2) * wheel_mass * (wheel_radius*wheel_radius)}" />
+            <mass value="2.8498940e-02" />
+            <inertia ixx="1.1175580e-05" ixy="-4.2369783e-11" ixz="-5.9381719e-09"
+                     iyy="1.1192413e-05" iyz="-1.4400107e-11"
+                     izz="2.0712558e-05" />
         </inertial>
     </link>
@@ -138,5 +134,5 @@
         <visual>
             <geometry>
-                <sphere radius="${caster_wheel_radius}"/>
+                <mesh filename="file://$(find robot_description)/urdf/left_tire_sim.stl" scale="0.0009 0.0009 0.0009"/>
             </geometry>
             <material name="white"/>
@@ -156,7 +152,7 @@
     </link>
     <gazebo reference="caster_wheel">
-        <material>Gazebo/White</material>
         <mu1 value="0.001"/>
         <mu2 value="0.001"/>
+        <material>Gazebo/White</material>
     </gazebo>
 </robot>
